Commit message: add franka_moveit_config

File: colcon_ws/src/franka_moveit_config/config/panda.ros2_control.xacro (robot description, xacro)
@@ -2,5 +2,5 @@
 <robot xmlns:xacro="http://www.ros.org/wiki/xacro">
     <xacro:macro name="panda_ros2_control" params="name initial_positions_file ros2_control_hardware_type">
-        <xacro:property name="initial_positions" value="${xacro.load_yaml(initial_positions_file)['initial_positions']}"/>
+        <xacro:property name="initial_positions" value="${load_yaml(initial_positions_file)['initial_positions']}"/>
         <ros2_control name="${name}" type="system">
             <hardware>
@@ -17,7 +17,5 @@
                   <param name="initial_value">${initial_positions['panda_joint1']}</param>
                 </state_interface>
-                <state_interface name="velocity">
-                  <param name="initial_value">0.0</param>
-                </state_interface>
+                <state_interface name="velocity"/>
                 <state_interface name="effort"/>
             </joint>
@@ -27,7 +25,5 @@
                   <param name="initial_value">${initial_positions['panda_joint2']}</param>
                 </state_interface>
-                <state_interface name="velocity">
-                  <param name="initial_value">0.0</param>
-                </state_interface>
+                <state_interface name="velocity"/>
                 <state_interface name="effort"/>
             </joint>
@@ -37,7 +33,5 @@
                   <param name="initial_value">${initial_positions['panda_joint3']}</param>
                 </state_interface>
-                <state_interface name="velocity">
-                  <param name="initial_value">0.0</param>
-                </state_interface>
+                <state_interface name="velocity"/>
                 <state_interface name="effort"/>
             </joint>
@@ -47,7 +41,5 @@
                   <param name="initial_value">${initial_positions['panda_joint4']}</param>
                 </state_interface>
-                <state_interface name="velocity">
-                  <param name="initial_value">0.0</param>
-                </state_interface>
+                <state_interface name="velocity"/>
                 <state_interface name="effort"/>
             </joint>
@@ -57,7 +49,5 @@
                   <param name="initial_value">${initial_positions['panda_joint5']}</param>
                 </state_interface>
-                <state_interface name="velocity">
-                  <param name="initial_value">0.0</param>
-                </state_interface>
+                <state_interface name="velocity"/>
                 <state_interface name="effort"/>
             </joint>
@@ -67,7 +57,5 @@
                   <param name="initial_value">${initial_positions['panda_joint6']}</param>
                 </state_interface>
-                <state_interface name="velocity">
-                  <param name="initial_value">0.0</param>
-                </state_interface>
+                <state_interface name="velocity"/>
                 <state_interface name="effort"/>
             </joint>
@@ -77,29 +65,13 @@
                   <param name="initial_value">${initial_positions['panda_joint7']}</param>
                 </state_interface>
-                <state_interface name="velocity">
-                  <param name="initial_value">0.0</param>
-                </state_interface>
+                <state_interface name="velocity"/>
                 <state_interface name="effort"/>
             </joint>
             <joint name="panda_finger_joint1">
-                <command_interface name="position" />
+                <command_interface name="position"/>
                 <state_interface name="position">
-                  <param name="initial_value">0.0</param>
+                  <param name="initial_value">${initial_positions['panda_finger_joint1']}</param>
                 </state_interface>
-                <state_interface name="velocity">
-                    <param name="initial_value">0.0</param>
-                </state_interface>
-                <state_interface name="effort"/>
-            </joint>
-            <joint name="panda_finger_joint2">
-                <param name="mimic">panda_finger_joint1</param>
-                <param name="multiplier">1</param>
-                <command_interface name="position" />
-                <state_interface name="position">
-                  <param name="initial_value">0.0</param>
-                </state_interface>
-                <state_interface name="velocity">
-                    <param name="initial_value">0.0</param>
-                </state_interface>
+                <state_interface name="velocity"/>
                 <state_interface name="effort"/>
             </joint>

File: colcon_ws/src/franka_moveit_config/config/panda.urdf.xacro (robot description, xacro)
@@ -5,6 +5,6 @@
     <!-- Import panda urdf file -->
     <xacro:include filename="$(find moveit_resources_panda_description)/urdf/panda.urdf" />
-    <!-- Import panda ros2_control description -->
+    <!-- Import control_xacro -->
     <xacro:include filename="panda.ros2_control.xacro" />
-    <xacro:panda_ros2_control name="panda" initial_positions_file="$(arg initial_positions_file)" ros2_control_hardware_type="$(arg ros2_control_hardware_type)"/>
+    <xacro:panda_ros2_control name="FakeSystem" initial_positions_file="$(arg initial_positions_file)" ros2_control_hardware_type="$(arg ros2_control_hardware_type)"/>
 </robot>
