Commit message: [add] SurfaceGripper support

File: colcon_ws/src/diffbot_description/isaac/diffbot.isaac.xacro (robot description, xacro)
@@ -48,4 +48,18 @@
         <update_rate>10</update_rate>
       </sensor>
+      <surface_gripper name="body_link">
+        <topic>gripper_enable</topic>
+        <offset_x>1.0</offset_x>
+        <offset_y>0</offset_y>
+        <offset_z>0</offset_z>
+        <axis>1 0 0</axis>
+        <grip_threshold>0.1</grip_threshold>
+        <force_limit>1.0e2</force_limit>
+        <torque_limit>1.0e3</torque_limit>
+        <bend_angle>0.7854</bend_angle>
+        <stiffness>1.0e4</stiffness>
+        <damping>1.0e3</damping>
+        <retry_close>False</retry_close>
+      </surface_gripper>
     </isaac>
   </xacro:macro>

Commit message: [update] ROS packages for Isaac Sim 5.2.0

File: colcon_ws/src/diffbot_description/isaac/diffbot.isaac.xacro (robot description, xacro)
@@ -64,4 +64,6 @@
       <thruster name="body_link">
       </thruster>
+      <thruster name="thruster_link">
+      </thruster>
     </isaac>
   </xacro:macro>

File: colcon_ws/src/diffbot_description/robots/diffbot_description.urdf.xacro (robot description, xacro)
@@ -149,4 +149,21 @@
     -->
   </link>
+  <joint name="thruster_joint" type="fixed">
+    <parent link="base_link"/>
+    <child  link="thruster_link"/>
+    <origin xyz="-0.1 0.1 0.1" rpy="0 ${pi/2} 0"/>
+  </joint>
+  <link name="thruster_link">
+    <!-- If visual tag is enable, camera's view is blocked. -->
+    <!--
+    <visual>
+      <origin xyz="0 0 0" rpy="0 -1.57 0" />
+      <geometry>
+        <cylinder radius="0.01" length="0.01" />
+      </geometry>
+      <material name="white" />
+    </visual>
+    -->
+  </link>
   </xacro:macro>
 </robot>
